Commit message: added joints training on tableworld

File: assets/robots/predefined/ur5/urdf/ur5_no_collision.urdf (robot description, URDF)
Before this commit: robot ur5_with_torch, 9 links, 8 joints
Links:
- link base_link: mass None -> 0.0
- link ee_link: mass None -> 0.2
- link forearm_link: mass None -> 2.275
- link shoulder_link: mass None -> 3.7
- link upper_arm_link: mass None -> 8.393
- link wrist_1_link: mass None -> 1.219
- link wrist_2_link: mass None -> 1.219
- link wrist_3_link: mass None -> 0.1879
